File: Board/board_autorouted_2_layers.brd (EAGLE design)
At the start: 68.6 x 53.3 mm, 19 parts, among them IC1 L293D

Commit message: Finished, and autorouted everything on 2 layers.
Parts:
- removed MOT1, MOT2: (no value), pinhead:1X02
- removed S1, S3: (no value), adafruit:B3F-40XX
- added MOT11, MOT12, MOT21, MOT22: (no value), pinhead:1X01
- moved THWHEEL2 154.6 mm to (68.6, 17.8)
- moved THWHEEL1 144.0 mm to (61.0, 17.8)
- moved R1 143.7 mm to (47.0, 29.2), turned to 90 degrees
- moved SW1 121.9 mm to (59.7, 29.2), turned to 180 degrees
- moved R2 112.6 mm to (27.9, 8.89)
- moved SW2 111.3 mm to (27.9, 19.1), turned to 270 degrees
- moved R3 111.0 mm to (43.2, 33.0), turned to 180 degrees
- moved SW3 98.8 mm to (48.3, 43.2), turned to 270 degrees
- moved ULTRA 92.2 mm to (71.1, 48.3), turned to 90 degrees
- moved BUZZ 90.9 mm to (64.8, 47.0), turned to 270 degrees
- moved SRVO 78.4 mm to (58.4, 48.3), turned to 90 degrees
- moved PHOTO 72.3 mm to (52.1, 17.8)
- moved ALIM 49.9 mm to (47.0, 11.4)
- moved IC1 19.0 mm to (29.2, 41.9)
Connections:
- new net N$24: PCB1.2, SW1.3
- net N$1: now also MOT11.1; no longer MOT1.2
- net N$2: now also MOT12.1; no longer MOT1.1
- net N$3: now also IC1.14, MOT21.1; no longer IC1.11, MOT2.2
- net N$4: now also IC1.11, MOT22.1; no longer IC1.14, MOT2.1
Routing:
- net +5V: track 0.00 -> 175.2 mm
- net N$19: track 0.00 -> 55.0 mm, vias 0 -> 1
- net N$10: track 0.00 -> 38.4 mm, vias 0 -> 1
- net N$5: track 0.00 -> 38.2 mm
- net N$7: track 0.00 -> 28.8 mm, vias 0 -> 1
- net N$24: track 0.00 -> 27.5 mm
- net N$6: track 0.00 -> 21.1 mm
- net N$12: track 0.00 -> 18.7 mm
- net N$11: track 0.00 -> 18.4 mm
- net N$9: track 0.00 -> 17.9 mm
- net N$23: track 0.00 -> 14.1 mm
- net N$8: track 0.00 -> 13.7 mm, vias 0 -> 1
- net N$22: track 0.00 -> 13.6 mm
- net N$15: track 0.00 -> 10.8 mm
- net N$16: track 0.00 -> 10.4 mm
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