File: Board/board.brd (EAGLE design)
At the start: 78.7 x 73.7 mm, 23 parts, among them IC1 L293D, U1 ARDUINOR3-BPLACE

Commit message: Board cleanup
Parts:
- BUZ: value (none) -> Ding
Connections:
- net N$19 renamed PIN4
- net N$23 renamed PIN5
- net N$24 renamed PIN2
- net N$5 renamed PINA1
- net N$6 renamed PINA0
Routing:
- net GND: track 42.2 -> 16.4 mm
Changed lines of the file:
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@@
 <element name="SND" library="pinhead" package="1X03" value="" x="82.55" y="64.135"/>
 <element name="SRV" library="pinhead" package="1X03/90" value="" x="57.15" y="64.77" rot="R90"/>
-<element name="BUZ" library="pinhead" package="1X02" value="" x="59.69" y="46.99" rot="R270"/>
+<element name="BUZ" library="pinhead" package="1X02" value="Ding" x="59.69" y="46.99" rot="R270"/>
 <element name="U1" library="adafruit" package="ARDUINOR3-BPLACE" value="ARDUINOR3-BPLACE" x="15.24" y="7.62"/>
 <element name="WHL1" library="pinhead" package="1X02" value="" x="71.12" y="16.51" rot="R180"/>
@@
 <wire x1="56.515" y1="10.16" x2="55.88" y2="10.16" width="0.4064" layer="16"/>
 <wire x1="26.67" y1="34.29" x2="29.21" y2="34.29" width="0.4064" layer="16"/>
-<wire x1="29.21" y1="34.29" x2="29.21" y2="40.64" width="0.4064" layer="16"/>
-<wire x1="29.21" y1="40.64" x2="29.845" y2="41.275" width="0.4064" layer="16"/>
-<wire x1="51.435" y1="63.1825" x2="46.6725" y2="63.1825" width="0.4064" layer="16"/>
-<wire x1="46.6725" y1="63.1825" x2="38.4175" y2="71.4375" width="0.4064" layer="16"/>
-<wire x1="52.959" y1="61.976" x2="51.435" y2="62.865" width="0.4064" layer="16"/>
-<wire x1="51.435" y1="62.865" x2="51.435" y2="63.1825" width="0.4064" layer="16"/>
 <wire x1="52.959" y1="52.7685" x2="53.086" y2="52.7685" width="0.4064" layer="16"/>
 <wire x1="53.086" y1="52.7685" x2="53.086" y2="61.849" width="0.4064" layer="16"/>
@@
 <contactref element="WHL1" pad="2"/>
 <contactref element="WHL2" pad="2"/>
-<contactref element="R6" pad="2"/>
 <contactref element="SND" pad="2"/>
 <contactref element="SRV" pad="2"/>
@@
 <wire x1="48.644525" y1="64.77" x2="60.96" y2="64.77" width="0.4064" layer="16"/>
 <wire x1="46.355" y1="67.31" x2="46.2788" y2="67.5894" width="0.4064" layer="16"/>
-<contactref element="PHS-R" pad="1"/>
-<contactref element="PHS-R" pad="3"/>
 <wire x1="53.34" y1="10.16" x2="53.34" y2="12.7" width="0.4064" layer="16"/>
 <wire x1="53.34" y1="12.7" x2="53.34" y2="16.51" width="0.4064" layer="16"/>
-<wire x1="65.405" y1="18.415" x2="62.865" y2="18.415" width="0.4064" layer="16"/>
 <wire x1="21.59" y1="31.75" x2="19.05" y2="34.29" width="0.4064" layer="16"/>
 <wire x1="21.59" y1="31.75" x2="32.339875" y2="31.75" width="0.4064" layer="16"/>
@@
 <wire x1="62.73095" y1="64.77" x2="60.96" y2="64.77" width="0.4064" layer="16"/>
 <wire x1="77.47" y1="41.275" x2="67.31" y2="51.435" width="0.4064" layer="16"/>
-<wire x1="57.15" y1="12.7" x2="62.865" y2="18.415" width="0.4064" layer="16"/>
 <wire x1="53.34" y1="12.7" x2="57.15" y2="12.7" width="0.4064" layer="16"/>
-<wire x1="53.34" y1="10.16" x2="36.83" y2="26.67" width="0.4064" layer="16"/>
+<wire x1="53.34" y1="10.16" x2="36.982" y2="26.518" width="0.4064" layer="16"/>
 <contactref element="S2" pad="2"/>
 <wire x1="70.2056" y1="38.6588" x2="74.8538" y2="38.6588" width="0.4064" layer="16"/>
@@
 <wire x1="70.485" y1="38.3794" x2="70.2056" y2="38.6588" width="0.4064" layer="16"/>
 <contactref element="S1" pad="1"/>
-<wire x1="36.982" y1="12.7" x2="36.982" y2="26.518" width="0.4064" layer="16"/>
 <wire x1="36.982" y1="26.518" x2="36.83" y2="26.67" width="0.4064" layer="16"/>
 <wire x1="77.47" y1="41.275" x2="82.55" y2="41.275" width="0.4064" layer="16"/>
@@
 <wire x1="82.55" y1="64.135" x2="82.55" y2="46.1518" width="0.4064" layer="16"/>
 <wire x1="82.55" y1="46.1518" x2="83.5406" y2="45.1612" width="0.4064" layer="16"/>
-<wire x1="65.405" y1="18.415" x2="67.945" y2="18.415" width="0.4064" layer="16"/>
 <wire x1="67.945" y1="18.415" x2="69.85" y2="16.51" width="0.4064" layer="16"/>
 <wire x1="69.85" y1="22.86" x2="69.85" y2="20.32" width="0.4064" layer="16"/>
 <wire x1="69.85" y1="20.32" x2="67.945" y2="18.415" width="0.4064" layer="16"/>
+<contactref element="PHS-R" pad="1"/>
+<contactref element="PHS-R" pad="3"/>
+<contactref element="R6" pad="2"/>
+<wire x1="36.982" y1="26.518" x2="36.982" y2="12.7" width="0.4064" layer="16"/>
+<wire x1="62.865" y1="18.415" x2="57.15" y2="12.7" width="0.4064" layer="16"/>
+<wire x1="62.865" y1="18.415" x2="65.405" y2="18.415" width="0.4064" layer="16"/>
+<wire x1="65.405" y1="18.415" x2="67.945" y2="18.415" width="0.4064" layer="16"/>
 </signal>
 <signal name="N$8">
@@
 <wire x1="63.5" y1="52.07" x2="63.5" y2="58.42" width="0.4064" layer="16"/>
 </signal>
-<signal name="N$19">
-<contactref element="S3" pad="3"/>
+<signal name="PIN4">
 <contactref element="U1" pad="D4"/>
 <wire x1="68.58" y1="58.42" x2="68.58" y2="67.264875" width="0.4064" layer="16"/>
 <wire x1="68.58" y1="67.264875" x2="64.089875" y2="71.755" width="0.4064" layer="16"/>
-<wire x1="64.089875" y1="71.755" x2="53.34" y2="71.755" width="0.4064" layer="16"/>
-<wire x1="53.34" y1="71.755" x2="52.7812" y2="72.1106" width="0.4064" layer="16"/>
+<wire x1="64.089875" y1="71.755" x2="53.1368" y2="71.755" width="0.4064" layer="16"/>
+<contactref element="S3" pad="3"/>
+<wire x1="52.7812" y1="72.1106" x2="53.1368" y2="71.755" width="0.4064" layer="16"/>
 </signal>
 <signal name="N$21">
@@
 <wire x1="31.75" y1="38.735" x2="31.75" y2="34.29" width="0.4064" layer="16"/>
 </signal>
-<signal name="N$24">
+<signal name="PIN2">
+<contactref element="U1" pad="D2"/>
+<wire x1="73.66" y1="50.8" x2="79.0194" y2="45.4406" width="0.4064" layer="16"/>
+<wire x1="73.66" y1="58.42" x2="73.66" y2="50.8" width="0.4064" layer="16"/>
 <contactref element="S1" pad="3"/>
-<contactref element="U1" pad="D2"/>
-<wire x1="73.66" y1="50.8" x2="78.74" y2="45.72" width="0.4064" layer="16"/>
-<wire x1="73.66" y1="58.42" x2="73.66" y2="50.8" width="0.4064" layer="16"/>
-<wire x1="78.74" y1="45.72" x2="79.0194" y2="45.1612" width="0.4064" layer="16"/>
+<wire x1="79.0194" y1="45.1612" x2="79.0194" y2="45.4406" width="0.4064" layer="16"/>
 </signal>
 <signal name="PIN13">
@@
 <contactref element="U1" pad="VIN"/>
 </signal>
-<signal name="N$6">
+<signal name="PINA0">
 <contactref element="U1" pad="A0"/>
+<wire x1="62.865" y1="13.335" x2="66.04" y2="10.16" width="0.4064" layer="16"/>
 <contactref element="PHS-R" pad="4"/>
-<wire x1="62.865" y1="15.875" x2="62.865" y2="13.335" width="0.4064" layer="16"/>
-<wire x1="62.865" y1="13.335" x2="66.04" y2="10.16" width="0.4064" layer="16"/>
+<wire x1="62.865" y1="13.335" x2="62.865" y2="15.875" width="0.4064" layer="16"/>
 </signal>
 <signal name="N$11">
@@
 <wire x1="76.048" y1="16.51" x2="72.39" y2="16.51" width="0.4064" layer="16"/>
 </signal>
-<signal name="N$5">
+<signal name="PINA1">
 <contactref element="U1" pad="A1"/>
+<wire x1="65.405" y1="13.335" x2="68.58" y2="10.16" width="0.4064" layer="16"/>
 <contactref element="PHS-R" pad="2"/>
 <wire x1="65.405" y1="15.875" x2="65.405" y2="13.335" width="0.4064" layer="16"/>
-<wire x1="65.405" y1="13.335" x2="68.58" y2="10.16" width="0.4064" layer="16"/>
 </signal>
 <signal name="N$13">
@@
 <wire x1="71.12" y1="61.845475" x2="71.12" y2="58.42" width="0.4064" layer="16"/>
 </signal>
-<signal name="N$23">
+<signal name="PIN5">
 <contactref element="U1" pad="D5"/>
+<wire x1="65.6844" y1="58.0644" x2="66.04" y2="58.42" width="0.4064" layer="16"/>
 <contactref element="S2" pad="3"/>
-<wire x1="65.6844" y1="45.1612" x2="65.6844" y2="58.0644" width="0.4064" layer="16"/>
-<wire x1="65.6844" y1="58.0644" x2="66.04" y2="58.42" width="0.4064" layer="16"/>
+<wire x1="65.6844" y1="58.0644" x2="65.6844" y2="45.1612" width="0.4064" layer="16"/>
 </signal>
 </signals>

Commit message: Board preparation
Parts:
- moved SND 31.3 mm to (52.1, 57.1)
- moved R1 28.2 mm to (50.8, 36.8)
- moved S1 28.0 mm to (53.3, 43.8)
- moved R4 27.3 mm to (50.2, 15.9)
- moved R5 26.4 mm to (50.2, 19.7), turned to 180 degrees
- moved BUZ 26.3 mm to (34.3, 40.0)
- moved SRV 26.3 mm to (31.8, 57.8)
- moved U1 26.3 mm to (-10.2, 0.64)
- moved R2 25.9 mm to (40.0, 36.8)
- moved ALIM 25.8 mm to (29.5, 10.8), turned to 0 degrees
- moved WHL2 25.6 mm to (45.7, 19.7)
- moved S2 25.5 mm to (42.5, 43.8)
- moved WHL1 25.4 mm to (45.7, 15.9)
- moved S3 24.0 mm to (28.6, 58.1)
- moved PHS-R 22.3 mm to (43.2, 9.53)
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Routing:
- net N$5: track 0.00 -> 122.6 mm
- net N$6: track 0.00 -> 116.2 mm
- net +5V: track 217.8 -> 156.5 mm
- net PIN13: track 63.7 -> 42.5 mm
- net N$7: track 44.5 -> 25.8 mm
- net N$10: track 65.5 -> 48.7 mm
- net GND: track 16.4 -> 32.1 mm
- net N$9: track 38.6 -> 23.4 mm
- net N$8: track 31.4 -> 16.3 mm
- net PIN12: track 60.0 -> 45.3 mm
- net PIN4: track 26.7 -> 16.2 mm
- net PIN2: track 15.5 -> 5.54 mm
- net PIN5: track 13.4 -> 4.52 mm
- net N$22: track 13.3 -> 8.18 mm
- net N$11: track 10.5 -> 15.0 mm
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Other:
- board size 78.7 x 73.7 mm -> 58.7 x 63.5 mm
